Commit message: fix: go2_description: utlidar joint

File: src/go2_description/urdf/go2.urdf (robot description, URDF)
Before this commit: robot go2, 33 links, 32 joints
Links:
- removed link radar
- added link utlidar, mass 0
Joints:
- removed joint radar_joint
- added joint utlidar_joint: type fixed, parent base_link, child utlidar, origin xyz=0.28945 0.032 -0.036825 rpy=0 2.8782 0, axis 0 0 0

Commit message: fix: go2_control: no deskewed cloud

File: src/go2_description/urdf/go2.urdf (robot description, URDF)
Before this commit: robot go2, 33 links, 32 joints
Joints:
- joint utlidar_joint: origin xyz=0.28945 0.032 -0.036825 rpy=0 2.8782 0 -> xyz=0.28945 0 -0.046825 rpy=0 2.8782 0
